File: PCB/ManPowerCharger.sch (KiCad schematic (older format))
At the start: 30 parts, among them J1 Conn_01x02_Male, J2 Conn_01x03_Male, Q1 2SJ681(Q), Q2 2SK4017(Q)

Commit message: 回路図修正（PCB未反映）
Parts:
- removed D2: LED, LED_THT:LED_D3.0mm, symbol Device:LED
- removed R2: 1k, Resistor_THT:R_Axial_DIN0204_L3.6mm_D1.6mm_P7.62mm_Horizontal, symbol Device:R
- added D?: D, Diode_THT:D_A-405_P7.62mm_Horizontal, symbol Device:D
Connections:
- net VBAT: now also D?.2 (A)
- net +12V renamed VCC
- net VCC: now also D?.1 (K)
Other:
- note added: "Power Supply\nAE-TPS7A4700"
- note removed: "Power Supply"
- moved on the sheet: J2, Q1, Q2, R1, R3, R4, R5, R6, R7, R8, R9
